Commit message: Update car_base.xacro

File: robot/urdf/car_base.xacro (robot description, xacro)
@@ -1,16 +1,16 @@
 <robot name="car_base" xmlns:xacro="http://www.ros.org/wiki/xacro">
-    <!-- 封装变量、常量 -->
+    <!-- 封装變量、常量 -->
     <xacro:property name="PI" value="3.1415926"/>
-    <!-- 宏:黑色设置 -->
+    <!-- 黑色 -->
     <material name="black">
         <color rgba="0.0 0.0 0.0 1.0" />
     </material>
-    <!-- 底盘属性 -->
-    <xacro:property name="base_footprint_radius" value="0.001" /> <!-- base_footprint 半径  -->
-    <xacro:property name="base_link_radius" value="0.1" />        <!-- base_link 半径 -->
-    <xacro:property name="base_link_length" value="0.08" />       <!-- base_link 长 -->
-    <xacro:property name="earth_space" value="0.015" />           <!-- 离地间距 -->
-    <xacro:property name="base_link_m" value="0.5" />             <!-- 质量  -->
-    <!-- 底盘 -->
+    <!-- 底盤属性 -->
+    <xacro:property name="base_footprint_radius" value="0.001" /> <!-- base_footprint radis  -->
+    <xacro:property name="base_link_radius" value="0.1" />        <!-- base_link rad -->
+    <xacro:property name="base_link_length" value="0.08" />       <!-- base_link 長 -->
+    <xacro:property name="earth_space" value="0.015" />           <!-- 離地高度 -->
+    <xacro:property name="base_link_m" value="0.5" />             <!-- weight  -->
+    <!-- 底盤 -->
     <link name="base_footprint">
         <visual>
@@ -46,10 +46,10 @@
         <material>Gazebo/Yellow</material>
     </gazebo>
-    <!-- 驱动轮 -->
-    <!-- 驱动轮属性 -->
-    <xacro:property name="wheel_radius" value="0.0325" /><!-- 半径 -->
-    <xacro:property name="wheel_length" value="0.015" /><!-- 宽度 -->
-    <xacro:property name="wheel_m" value="0.05" /> <!-- 质量  -->
-    <!-- 驱动轮宏实现 -->
+    <!--驅動倫倫 -->
+    <!-- 驅動輪属性 -->
+    <xacro:property name="wheel_radius" value="0.0325" /><!-- rad -->
+    <xacro:property name="wheel_length" value="0.015" /><!-- 寬 -->
+    <xacro:property name="wheel_m" value="0.05" /> <!-- weight  -->
+    <!-- 驅動輪Macro -->
     <xacro:macro name="add_wheels" params="name flag">
         <link name="${name}_wheel">
@@ -64,26 +64,5 @@
                 <geometry>
                     <cylinder radius="${wheel_radius}" length="${wheel_length}" />
-                </geometry>
-                <origin xyz="0.0 0.0 0.0" rpy="${PI / 2} 0.0 0.0" />
-            </collision>
-            <xacro:cylinder_inertial_matrix m="${wheel_m}" r="${wheel_radius}" h="${wheel_length}" />
-        </link>
-      <joint name="${name}_wheel2base_link" type="continuous">
-          <parent link="base_link" />
-          <child link="${name}_wheel" />
-          <origin xyz="0 ${flag * base_link_radius} ${-(earth_space + base_link_length / 2 - wheel_radius) }" />
-          <axis xyz="0 1 0" />
-      </joint>
-      <gazebo reference="${name}_wheel">
-          <material>Gazebo/Red</material>
-      </gazebo>
-    </xacro:macro>
-    <xacro:add_wheels name="left" flag="1" />
-    <xacro:add_wheels name="right" flag="-1" />
-    <!-- 支撑轮 -->
-    <!-- 支撑轮属性 -->
-    <xacro:property name="support_wheel_radius" value="0.0075" /> <!-- 支撑轮半径 -->
-    <xacro:property name="support_wheel_m" value="0.03" /> <!-- 质量  -->
-    <!-- 支撑轮宏 -->
+                </輔助輪macro -->
     <xacro:macro name="add_support_wheel" params="name flag" >
         <link name="${name}_wheel">

Commit message: Update car_base.xacro

File: robot/urdf/car_base.xacro (robot description, xacro)
@@ -1,16 +1,16 @@
 <robot name="car_base" xmlns:xacro="http://www.ros.org/wiki/xacro">
-    <!-- 封装變量、常量 -->
+    <!-- 封装变量、常量 -->
     <xacro:property name="PI" value="3.1415926"/>
-    <!-- 黑色 -->
+    <!-- 宏:黑色设置 -->
     <material name="black">
         <color rgba="0.0 0.0 0.0 1.0" />
     </material>
-    <!-- 底盤属性 -->
-    <xacro:property name="base_footprint_radius" value="0.001" /> <!-- base_footprint radis  -->
-    <xacro:property name="base_link_radius" value="0.1" />        <!-- base_link rad -->
-    <xacro:property name="base_link_length" value="0.08" />       <!-- base_link 長 -->
-    <xacro:property name="earth_space" value="0.015" />           <!-- 離地高度 -->
-    <xacro:property name="base_link_m" value="0.5" />             <!-- weight  -->
-    <!-- 底盤 -->
+    <!-- 底盘属性 -->
+    <xacro:property name="base_footprint_radius" value="0.001" /> <!-- base_footprint 半径  -->
+    <xacro:property name="base_link_radius" value="0.1" />        <!-- base_link 半径 -->
+    <xacro:property name="base_link_length" value="0.08" />       <!-- base_link 长 -->
+    <xacro:property name="earth_space" value="0.015" />           <!-- 离地间距 -->
+    <xacro:property name="base_link_m" value="0.5" />             <!-- 质量  -->
+    <!-- 底盘 -->
     <link name="base_footprint">
         <visual>
@@ -46,10 +46,10 @@
         <material>Gazebo/Yellow</material>
     </gazebo>
-    <!--驅動倫倫 -->
-    <!-- 驅動輪属性 -->
-    <xacro:property name="wheel_radius" value="0.0325" /><!-- rad -->
-    <xacro:property name="wheel_length" value="0.015" /><!-- 寬 -->
-    <xacro:property name="wheel_m" value="0.05" /> <!-- weight  -->
-    <!-- 驅動輪Macro -->
+    <!-- 驱动轮 -->
+    <!-- 驱动轮属性 -->
+    <xacro:property name="wheel_radius" value="0.0325" /><!-- 半径 -->
+    <xacro:property name="wheel_length" value="0.015" /><!-- 宽度 -->
+    <xacro:property name="wheel_m" value="0.05" /> <!-- 质量  -->
+    <!-- 驱动轮宏实现 -->
     <xacro:macro name="add_wheels" params="name flag">
         <link name="${name}_wheel">
@@ -64,5 +64,26 @@
                 <geometry>
                     <cylinder radius="${wheel_radius}" length="${wheel_length}" />
-                </輔助輪macro -->
+                </geometry>
+                <origin xyz="0.0 0.0 0.0" rpy="${PI / 2} 0.0 0.0" />
+            </collision>
+            <xacro:cylinder_inertial_matrix m="${wheel_m}" r="${wheel_radius}" h="${wheel_length}" />
+        </link>
+      <joint name="${name}_wheel2base_link" type="continuous">
+          <parent link="base_link" />
+          <child link="${name}_wheel" />
+          <origin xyz="0 ${flag * base_link_radius} ${-(earth_space + base_link_length / 2 - wheel_radius) }" />
+          <axis xyz="0 1 0" />
+      </joint>
+      <gazebo reference="${name}_wheel">
+          <material>Gazebo/Red</material>
+      </gazebo>
+    </xacro:macro>
+    <xacro:add_wheels name="left" flag="1" />
+    <xacro:add_wheels name="right" flag="-1" />
+    <!-- 支撑轮 -->
+    <!-- 支撑轮属性 -->
+    <xacro:property name="support_wheel_radius" value="0.0075" /> <!-- 支撑轮半径 -->
+    <xacro:property name="support_wheel_m" value="0.03" /> <!-- 质量  -->
+    <!-- 支撑轮宏 -->
     <xacro:macro name="add_support_wheel" params="name flag" >
         <link name="${name}_wheel">

Commit message: Update car_base.xacro

File: robot/urdf/car_base.xacro (robot description, xacro)
@@ -1,16 +1,16 @@
 <robot name="car_base" xmlns:xacro="http://www.ros.org/wiki/xacro">
-    <!-- 封装变量、常量 -->
+    <!-- 封装變量、常量 -->
     <xacro:property name="PI" value="3.1415926"/>
-    <!-- 宏:黑色设置 -->
+    <!-- macro:黑色 -->
     <material name="black">
         <color rgba="0.0 0.0 0.0 1.0" />
     </material>
-    <!-- 底盘属性 -->
-    <xacro:property name="base_footprint_radius" value="0.001" /> <!-- base_footprint 半径  -->
-    <xacro:property name="base_link_radius" value="0.1" />        <!-- base_link 半径 -->
-    <xacro:property name="base_link_length" value="0.08" />       <!-- base_link 长 -->
-    <xacro:property name="earth_space" value="0.015" />           <!-- 离地间距 -->
-    <xacro:property name="base_link_m" value="0.5" />             <!-- 质量  -->
-    <!-- 底盘 -->
+    <!-- 底盤属性 -->
+    <xacro:property name="base_footprint_radius" value="0.001" /> <!-- base_footprint radis  -->
+    <xacro:property name="base_link_radius" value="0.1" />        <!-- base_link rad -->
+    <xacro:property name="base_link_length" value="0.08" />       <!-- base_link 長 -->
+    <xacro:property name="earth_space" value="0.015" />           <!-- 離地高度 -->
+    <xacro:property name="base_link_m" value="0.5" />             <!-- weight  -->
+    <!-- 底盤 -->
     <link name="base_footprint">
         <visual>
@@ -46,10 +46,10 @@
         <material>Gazebo/Yellow</material>
     </gazebo>
-    <!-- 驱动轮 -->
-    <!-- 驱动轮属性 -->
-    <xacro:property name="wheel_radius" value="0.0325" /><!-- 半径 -->
-    <xacro:property name="wheel_length" value="0.015" /><!-- 宽度 -->
-    <xacro:property name="wheel_m" value="0.05" /> <!-- 质量  -->
-    <!-- 驱动轮宏实现 -->
+    <!-- 驅動倫 -->
+    <!-- 驅動倫属性 -->
+    <xacro:property name="wheel_radius" value="0.0325" /><!-- rad -->
+    <xacro:property name="wheel_length" value="0.015" /><!-- 寬 -->
+    <xacro:property name="wheel_m" value="0.05" /> <!-- weight  -->
+    <!-- 驅動倫macro -->
     <xacro:macro name="add_wheels" params="name flag">
         <link name="${name}_wheel">
@@ -81,9 +81,9 @@
     <xacro:add_wheels name="left" flag="1" />
     <xacro:add_wheels name="right" flag="-1" />
-    <!-- 支撑轮 -->
-    <!-- 支撑轮属性 -->
-    <xacro:property name="support_wheel_radius" value="0.0075" /> <!-- 支撑轮半径 -->
-    <xacro:property name="support_wheel_m" value="0.03" /> <!-- 质量  -->
-    <!-- 支撑轮宏 -->
+    <!-- 輔助輪 -->
+    <!-- 輔助輪属性 -->
+    <xacro:property name="support_wheel_radius" value="0.0075" /> <!-- 輔助輪radis -->
+    <xacro:property name="support_wheel_m" value="0.03" /> <!-- weight  -->
+    <!-- macro -->
     <xacro:macro name="add_support_wheel" params="name flag" >
         <link name="${name}_wheel">

Commit message: Update car_base.xacro

File: robot/urdf/car_base.xacro (robot description, xacro)
@@ -1,16 +1,16 @@
 <robot name="car_base" xmlns:xacro="http://www.ros.org/wiki/xacro">
-    <!-- 封装變量、常量 -->
+    <!-- Encapsulating variables and constants -->
     <xacro:property name="PI" value="3.1415926"/>
-    <!-- macro:黑色 -->
+    <!-- Macro: black material -->
     <material name="black">
         <color rgba="0.0 0.0 0.0 1.0" />
     </material>
-    <!-- 底盤属性 -->
-    <xacro:property name="base_footprint_radius" value="0.001" /> <!-- base_footprint radis  -->
-    <xacro:property name="base_link_radius" value="0.1" />        <!-- base_link rad -->
-    <xacro:property name="base_link_length" value="0.08" />       <!-- base_link 長 -->
-    <xacro:property name="earth_space" value="0.015" />           <!-- 離地高度 -->
-    <xacro:property name="base_link_m" value="0.5" />             <!-- weight  -->
-    <!-- 底盤 -->
+    <!-- Chassis properties -->
+    <xacro:property name="base_footprint_radius" value="0.001" /> <!-- Base footprint radius -->
+    <xacro:property name="base_link_radius" value="0.1" />        <!-- Base link radius -->
+    <xacro:property name="base_link_length" value="0.08" />       <!-- Base link length -->
+    <xacro:property name="earth_space" value="0.015" />           <!-- Ground clearance -->
+    <xacro:property name="base_link_m" value="0.5" />             <!-- Weight -->
+    <!-- Chassis -->
     <link name="base_footprint">
         <visual>
@@ -41,15 +41,15 @@
         <parent link="base_footprint" />
         <child link="base_link" />
-        <origin xyz="0 0 ${earth_space + base_link_length / 2 }" />
+        <origin xyz="0 0 ${earth_space + base_link_length / 2}" />
     </joint>
     <gazebo reference="base_link">
         <material>Gazebo/Yellow</material>
     </gazebo>
-    <!-- 驅動倫 -->
-    <!-- 驅動倫属性 -->
-    <xacro:property name="wheel_radius" value="0.0325" /><!-- rad -->
-    <xacro:property name="wheel_length" value="0.015" /><!-- 寬 -->
-    <xacro:property name="wheel_m" value="0.05" /> <!-- weight  -->
-    <!-- 驅動倫macro -->
+    <!-- Drive wheels -->
+    <!-- Drive wheel properties -->
+    <xacro:property name="wheel_radius" value="0.0325" /> <!-- Radius -->
+    <xacro:property name="wheel_length" value="0.015" />  <!-- Width -->
+    <xacro:property name="wheel_m" value="0.05" />       <!-- Weight -->
+    <!-- Drive wheel macro -->
     <xacro:macro name="add_wheels" params="name flag">
         <link name="${name}_wheel">
@@ -69,22 +69,22 @@
             <xacro:cylinder_inertial_matrix m="${wheel_m}" r="${wheel_radius}" h="${wheel_length}" />
         </link>
-      <joint name="${name}_wheel2base_link" type="continuous">
-          <parent link="base_link" />
-          <child link="${name}_wheel" />
-          <origin xyz="0 ${flag * base_link_radius} ${-(earth_space + base_link_length / 2 - wheel_radius) }" />
-          <axis xyz="0 1 0" />
-      </joint>
-      <gazebo reference="${name}_wheel">
-          <material>Gazebo/Red</material>
-      </gazebo>
+        <joint name="${name}_wheel2base_link" type="continuous">
+            <parent link="base_link" />
+            <child link="${name}_wheel" />
+            <origin xyz="0 ${flag * base_link_radius} ${-(earth_space + base_link_length / 2 - wheel_radius)}" />
+            <axis xyz="0 1 0" />
+        </joint>
+        <gazebo reference="${name}_wheel">
+            <material>Gazebo/Red</material>
+        </gazebo>
     </xacro:macro>
     <xacro:add_wheels name="left" flag="1" />
     <xacro:add_wheels name="right" flag="-1" />
-    <!-- 輔助輪 -->
-    <!-- 輔助輪属性 -->
-    <xacro:property name="support_wheel_radius" value="0.0075" /> <!-- 輔助輪radis -->
-    <xacro:property name="support_wheel_m" value="0.03" /> <!-- weight  -->
-    <!-- macro -->
-    <xacro:macro name="add_support_wheel" params="name flag" >
+    <!-- Support wheels -->
+    <!-- Support wheel properties -->
+    <xacro:property name="support_wheel_radius" value="0.0075" /> <!-- Support wheel radius -->
+    <xacro:property name="support_wheel_m" value="0.03" />       <!-- Weight -->
+    <!-- Support wheel macro -->
+    <xacro:macro name="add_support_wheel" params="name flag">
         <link name="${name}_wheel">
             <visual>
